Commit message: 💥 Add mini sumo meshes and urdf
Co-authored-by: Guigo62 <Guigo62@users.noreply.github.com>

File: urdf/mini_sumo.urdf (robot description, URDF)
Before this commit: robot mini_sumo, 4 links, 3 joints
Links:
- removed link imu_link
- link base_link: mass 0.0297313079671725 -> 0.384905526771832; geometry collision mesh filename=package://sumo_simulation/meshes/base_link_collision.STL; visual mesh filename=package://sumo_simulation/meshes/base_link_visual.STL
- link left_wheel_link: mass 0.0293925354796172 -> 0.051954; geometry collision cylinder length=25e-3 radius=17.5e-3; visual cylinder length=25e-3 radius=17.5e-3
- link right_wheel_link: mass 0.0293925354796178 -> 0.051954; geometry collision cylinder length=25e-3 radius=17.5e-3; visual cylinder length=25e-3 radius=17.5e-3
Joints:
- removed joint imu_joint
- joint left_wheel_joint: axis 0 1 0 -> 0 0 -1; origin xyz=0 0.0755 0 rpy=0 0 0 -> xyz=-0.0365 0.0375 0.0125 rpy=1.5708 0 0
- joint right_wheel_joint: axis 0 1 0 -> 0 0 1; origin xyz=0 -0.076 0 rpy=0 0 0 -> xyz=-0.0365 -0.0375 0.0125 rpy=-1.5708 0 0

Commit message: ✨ Add distance sensor to model

File: urdf/mini_sumo.urdf (robot description, URDF)
Before this commit: robot montagem_sumo_padrao, 3 links, 2 joints
Links:
- added link ds0_link
- added link ds1_link
- added link ds2_link
Joints:
- added joint ds0_joint: type fixed, parent base_link, child ds0_link, origin xyz=25e-3 25e-3 20e-3 rpy=0 -0.08 0.4, axis 0 0 0
- added joint ds1_joint: type fixed, parent base_link, child ds1_link, origin xyz=25e-3 0 20e-3 rpy=0 -0.08 0, axis 0 0 0
- added joint ds2_joint: type fixed, parent base_link, child ds2_link, origin xyz=25e-3 -25e-3 20e-3 rpy=0 -0.08 -0.4, axis 0 0 0

Commit message: 💄 Add distance sensors visual

File: urdf/mini_sumo.urdf (robot description, URDF)
Before this commit: robot montagem_sumo_padrao, 6 links, 5 joints
Links:
- link ds0_link: geometry visual box size=5e-3 5e-3 5e-3
- link ds1_link: geometry visual box size=5e-3 5e-3 5e-3
- link ds2_link: geometry visual box size=5e-3 5e-3 5e-3

Commit message: ✨ Add imu link visual

File: urdf/mini_sumo.urdf (robot description, URDF)
Before this commit: robot montagem_sumo_padrao, 6 links, 5 joints
Links:
- added link imu_link; visual box size=0.01 0.01 0.005
Joints:
- added joint imu_joint: type fixed, parent base_link, child imu_link, origin xyz=-35e-3 0 30e-3 rpy=0 0 0, axis 0 0 0

Commit message: 🚚 Rename distance sensors topics, links and joints

File: urdf/mini_sumo.urdf (robot description, URDF)
Before this commit: robot montagem_sumo_padrao, 7 links, 6 joints
Links:
- removed link ds0_link
- removed link ds1_link
- removed link ds2_link
- added link distance_sensor_0_link; visual box size=5e-3 5e-3 5e-3
- added link distance_sensor_1_link; visual box size=5e-3 5e-3 5e-3
- added link distance_sensor_2_link; visual box size=5e-3 5e-3 5e-3
Joints:
- removed joint ds0_joint
- removed joint ds1_joint
- removed joint ds2_joint
- added joint distance_sensor_0_joint: type fixed, parent base_link, child distance_sensor_0_link, origin xyz=25e-3 25e-3 20e-3 rpy=0 -0.08 0.4, axis 0 0 0
- added joint distance_sensor_1_joint: type fixed, parent base_link, child distance_sensor_1_link, origin xyz=25e-3 0 20e-3 rpy=0 -0.08 0, axis 0 0 0
- added joint distance_sensor_2_joint: type fixed, parent base_link, child distance_sensor_2_link, origin xyz=25e-3 -25e-3 20e-3 rpy=0 -0.08 -0.4, axis 0 0 0

Commit message: ✨ Create line sensor links and add plugin to .gazebo file

File: urdf/mini_sumo.urdf (robot description, URDF)
Before this commit: robot montagem_sumo_padrao, 7 links, 6 joints
Links:
- added link left_line_sensor_link; visual box size=1e-3 1e-3 1e-3
- added link right_line_sensor_link; visual box size=1e-3 1e-3 1e-3
Joints:
- added joint left_line_sensor_joint: type fixed, parent base_link, child left_line_sensor_link, origin xyz=40e-3 42.5e-3 2e-3 rpy=0 1.5708 0, axis 0 0 0
- added joint right_line_sensor_joint: type fixed, parent base_link, child right_line_sensor_link, origin xyz=40e-3 -42.5e-3 2e-3 rpy=0 1.5708 0, axis 0 0 0
